File: TR-808_Clone/Kicad/TR-808_clone/CTRL.sch (KiCad schematic (older format))
At the start: 185 parts, among them J30 Terminal, P10 Conn_02x03_Odd_Even, P11 Conn_02x03_Odd_Even, P12 Conn_02x03_Odd_Even, P13 Conn_02x03_Odd_Even, P14 Conn_02x03_Odd_Even, P15 Conn_02x03_Odd_Even, Q300 2SA733, Q301 2SA733, Q302 2SA733, Q303 2SA733, Q304 2SA733, Q305 2SA733, Q306 2SA733, Q307 2SA733, Q308 2SA733, Q309 2SA733, Q310 2SA733, Q311 2SA733, Q312 2SA733, Q313 2SA733, Q314 2SA733, Q315 2SA733, SW1 SW_DPDT_x2, SW2 SW_Push, SW3 SW_Push, SW4 SW_DPDT_x2, U30 74HC04, U31 BH2226F, U32 BH2226F, U33 TL084, U34 TL084, U35 TL084, U36 TL084

Commit message: Add files via upload
Parts:
- added C205: 0.1uF, Capacitor_THT:C_Disc_D3.4mm_W2.1mm_P2.50mm, symbol Device:C
Connections:
- net +5V: now also C205.1
- net GND: now also C205.2
Other:
- moved on the sheet: C200
Changed lines of the file:
@@
 L Device:C C?
 U 1 1 5D84376D
-P 3850 4500
+P 4250 4500
 AR Path="/5D76191B/5D84376D" Ref="C?"  Part="1"
 AR Path="/5D7620E2/5D84376D" Ref="C200"  Part="1"
-F 0 "C200" H 3965 4546 50  0000 L CNN
-F 1 "0.1uF" H 3965 4455 50  0000 L CNN
-F 2 "Capacitor_THT:C_Disc_D3.4mm_W2.1mm_P2.50mm" H 3888 4350 50  0001 C CNN
-F 3 "~" H 3850 4500 50  0001 C CNN
-	1    3850 4500
+F 0 "C200" H 4365 4546 50  0000 L CNN
+F 1 "0.1uF" H 4365 4455 50  0000 L CNN
+F 2 "Capacitor_THT:C_Disc_D3.4mm_W2.1mm_P2.50mm" H 4288 4350 50  0001 C CNN
+F 3 "~" H 4250 4500 50  0001 C CNN
+	1    4250 4500
 	1    0    0    -1
 $EndComp
@@
 L power:GND #PWR?
 U 1 1 5D843774
-P 3850 4700
+P 4250 4750
 AR Path="/5D76191B/5D843774" Ref="#PWR?"  Part="1"
 AR Path="/5D7620E2/5D843774" Ref="#PWR0443"  Part="1"
-F 0 "#PWR0443" H 3850 4450 50  0001 C CNN
-F 1 "GND" H 3855 4527 50  0000 C CNN
-F 2 "" H 3850 4700 50  0001 C CNN
-F 3 "" H 3850 4700 50  0001 C CNN
-	1    3850 4700
+F 0 "#PWR0443" H 4250 4500 50  0001 C CNN
+F 1 "GND" H 4255 4577 50  0000 C CNN
+F 2 "" H 4250 4750 50  0001 C CNN
+F 3 "" H 4250 4750 50  0001 C CNN
+	1    4250 4750
 	-1   0    0    -1
 $EndComp
 Wire Wire Line
-	3850 4650 3850 4700
+	4250 4650 4250 4700
 Text GLabel 1550 2700 0    50   Input ~ 0
 MIDI_IN_ESP32
@@
 L power:+5V #PWR?
 U 1 1 5D843816
-P 3850 4200
+P 4250 4200
 AR Path="/5D76191B/5D843816" Ref="#PWR?"  Part="1"
 AR Path="/5D7620E2/5D843816" Ref="#PWR0447"  Part="1"
-F 0 "#PWR0447" H 3850 4050 50  0001 C CNN
-F 1 "+5V" H 3865 4373 50  0000 C CNN
-F 2 "" H 3850 4200 50  0001 C CNN
-F 3 "" H 3850 4200 50  0001 C CNN
-	1    3850 4200
+F 0 "#PWR0447" H 4250 4050 50  0001 C CNN
+F 1 "+5V" H 4265 4373 50  0000 C CNN
+F 2 "" H 4250 4200 50  0001 C CNN
+F 3 "" H 4250 4200 50  0001 C CNN
+	1    4250 4200
 	1    0    0    -1
 $EndComp
 Wire Wire Line
-	3850 4200 3850 4250
+	4250 4200 4250 4250
 Text GLabel 6200 2800 2    50   Input ~ 0
 DA_BD
@@
 Connection ~ 2400 3050
 Wire Wire Line
-	3850 4250 3650 4250
+	4250 4250 4000 4250
 Wire Wire Line
-	3850 4250 3850 4350
-Connection ~ 3850 4250
+	4250 4250 4250 4350
+Connection ~ 4250 4250
 Connection ~ 1700 2850
 Wire Wire Line
@@
 	1    0    0    -1
 $EndComp
+$Comp
+L Device:C C?
+U 1 1 5E2C13D6
+P 4000 4500
+AR Path="/5D76191B/5E2C13D6" Ref="C?"  Part="1"
+AR Path="/5D7620E2/5E2C13D6" Ref="C205"  Part="1"
+F 0 "C205" H 4115 4546 50  0000 L CNN
+F 1 "0.1uF" H 4115 4455 50  0000 L CNN
+F 2 "Capacitor_THT:C_Disc_D3.4mm_W2.1mm_P2.50mm" H 4038 4350 50  0001 C CNN
+F 3 "~" H 4000 4500 50  0001 C CNN
+	1    4000 4500
+	-1   0    0    -1
+$EndComp
+Wire Wire Line
+	4000 4350 4000 4250
+Connection ~ 4000 4250
+Wire Wire Line
+	4000 4250 3650 4250
+Wire Wire Line
+	4000 4650 4000 4700
+Wire Wire Line
+	4000 4700 4250 4700
+Connection ~ 4250 4700
+Wire Wire Line
+	4250 4700 4250 4750
 $EndSCHEMATC
